Commit message: Set up ROS workspace in Orin

File: catkin_ws/src/mycobot_ros/mycobot_description/urdf/mycobot/mycobot_arm_realsense_urdf.urdf (robot description, URDF)
Before this commit: robot firefighter, 9 links, 8 joints
Links:
- link camera_depth_frame: geometry collision box size=0.025 0.025 0.025; visual box size=0.025 0.025 0.025

Commit message: Added *.dae model realsense & realsense camera to robot urdf

File: catkin_ws/src/mycobot_ros/mycobot_description/urdf/mycobot/mycobot_arm_realsense_urdf.urdf (robot description, URDF)
Before this commit: robot firefighter, 9 links, 8 joints
Links:
- added link base_link
- link camera_depth_frame: geometry 
- link camera_link: geometry collision mesh filename=package://mycobot_description/urdf/mycobot/realsense_d435.d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; visual mesh filename=package://mycobot_description/urdf/mycobot/realsense_d435.d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
Joints:
- removed joint joint1_to_camera_link
- added joint camera_link_to_base_link: type fixed, parent base_link, child camera_link, origin xyz=-0.3 0.0 0.5 rpy=2.0944 0.0 1.5708
- added joint joint1_to_base_link: type fixed, parent base_link, child joint1, origin xyz=0.0 0.0 0.0 rpy=0.0 0.0 0.0
- joint camera_depth_frame_to_camera_link: origin xyz=-0.1 0.05 0.1 rpy=0 0 1.5708 -> xyz=0.0 0.0 0.0 rpy=0.0 0.0 3.14

File: catkin_ws/src/realsense-ros/realsense2_description/urdf/test_d435_camera.urdf.xacro (robot description, xacro)
@@ -7,5 +7,5 @@
   <link name="base_link" />
   <xacro:sensor_d435 parent="base_link" use_nominal_extrinsics="$(arg use_nominal_extrinsics)" add_plug="$(arg add_plug)" use_mesh="$(arg use_mesh)">
-    <origin xyz="0 0 0" rpy="0 0 0"/>
+    <origin xyz="-0.3 0.5 0" rpy="0 0 0"/>
   </xacro:sensor_d435>
 </robot>

Commit message: Added stand to urdf model and test with mycobot_280jn

File: catkin_ws/src/mycobot_ros/mycobot_description/urdf/mycobot/mycobot_arm_realsense_urdf.urdf (robot description, URDF)
Before this commit: robot firefighter, 10 links, 9 joints
Links:
- added link stand_link; collision mesh filename=package://mycobot_description/urdf/mycobot/stand.dae; visual mesh filename=package://mycobot_description/urdf/mycobot/stand.dae
Joints:
- added joint stand_link_to_base_link: type fixed, parent base_link, child stand_link, origin xyz=-0.05 0.1 -0.07 rpy=1.5708 0.0 -1.5708
- joint camera_link_to_base_link: origin xyz=-0.3 0.0 0.5 rpy=2.0944 0.0 1.5708 -> xyz=-0.275 0.0 0.5 rpy=2.0944 0.0 1.5708

Commit message: Corrected frame TFs for depth camera in URDF model

File: catkin_ws/src/mycobot_ros/mycobot_description/urdf/mycobot/mycobot_arm_realsense_urdf.urdf (robot description, URDF)
Before this commit: robot firefighter, 11 links, 10 joints
Links:
- removed link camera_depth_frame
Joints:
- removed joint camera_depth_frame_to_camera_link
- joint camera_link_to_base_link: origin xyz=-0.275 0.0 0.5 rpy=2.0944 0.0 1.5708 -> xyz=-0.275 0.0 0.5 rpy=0.0 0.523599 0.0
